Commit message: Load EEF geom params and origin pose from yaml

File: xarm_description/urdf/other/other_geometry.urdf.xacro (robot description, xacro)
@@ -15,4 +15,6 @@
     geometry_mesh_origin_xyz:='0 0 0'
     geometry_mesh_origin_rpy:='0 0 0'
+    geometry_origin_xyz:='auto'
+    geometry_origin_rpy:='auto'
     geometry_mesh_tcp_xyz:='0 0 0'
     geometry_mesh_tcp_rpy:='0 0 0'
@@ -40,6 +42,19 @@
         <xacro:property name="_tcp_z" value="${geometry_radius * 2}"/>
       </xacro:unless>
-      <xacro:property name="_origin_xyz" value="0 0 ${_origin_y}"/>
-      <xacro:property name="_origin_rpy" value="0 0 0"/>
+      <xacro:property name="_auto_origin_xyz" value="0 0 ${_origin_y}"/>
+      <xacro:property name="_auto_origin_rpy" value="0 0 0"/>
+      <xacro:if value="${geometry_origin_xyz == 'auto'}">
+        <xacro:property name="_origin_xyz" value="${_auto_origin_xyz}"/>
+        <xacro:property name="_origin_rpy" value="${_auto_origin_rpy}"/>
+      </xacro:if>
+      <xacro:unless value="${geometry_origin_xyz == 'auto'}">
+        <xacro:property name="_origin_xyz" value="${geometry_origin_xyz}"/>
+        <xacro:if value="${geometry_origin_rpy == 'auto'}">
+          <xacro:property name="_origin_rpy" value="0 0 0"/>
+        </xacro:if>
+        <xacro:unless value="${geometry_origin_rpy == 'auto'}">
+          <xacro:property name="_origin_rpy" value="${geometry_origin_rpy}"/>
+        </xacro:unless>
+      </xacro:unless>
       <xacro:property name="_tcp_xyz" value="0 0 ${_tcp_z}"/>
       <xacro:property name="_tcp_rpy" value="0 0 0"/>

File: xarm_description/urdf/xarm_device.urdf.xacro (robot description, xacro)
@@ -30,4 +30,8 @@
   <xacro:arg name="geometry_mesh_origin_xyz" default="0 0 0"/>
   <xacro:arg name="geometry_mesh_origin_rpy" default="0 0 0"/>
+  <xacro:arg name="geometry_origin_xyz" default="auto"/>
+  <xacro:arg name="geometry_origin_rpy" default="auto"/>
+  <xacro:arg name="joint_eef_origin_xyz" default="0 0 0"/>
+  <xacro:arg name="joint_eef_origin_rpy" default="0 0 0"/>
   <xacro:arg name="geometry_mesh_tcp_xyz" default="0 0 0"/>
   <xacro:arg name="geometry_mesh_tcp_rpy" default="0 0 0"/>
@@ -55,4 +59,6 @@
     geometry_mesh_filename="$(arg geometry_mesh_filename)"
     geometry_mesh_origin_xyz="$(arg geometry_mesh_origin_xyz)" geometry_mesh_origin_rpy="$(arg geometry_mesh_origin_rpy)"
+    geometry_origin_xyz="$(arg geometry_origin_xyz)" geometry_origin_rpy="$(arg geometry_origin_rpy)"
+    joint_eef_origin_xyz="$(arg joint_eef_origin_xyz)" joint_eef_origin_rpy="$(arg joint_eef_origin_rpy)"
     geometry_mesh_tcp_xyz="$(arg geometry_mesh_tcp_xyz)" geometry_mesh_tcp_rpy="$(arg geometry_mesh_tcp_rpy)"
     robot_ip="$(arg robot_ip)" report_type="$(arg report_type)"

File: xarm_description/urdf/xarm_device_macro.xacro (robot description, xacro)
@@ -32,4 +32,8 @@
     geometry_mesh_origin_xyz:='0 0 0'
     geometry_mesh_origin_rpy:='0 0 0'
+    geometry_origin_xyz:='auto'
+    geometry_origin_rpy:='auto'
+    joint_eef_origin_xyz:='0 0 0'
+    joint_eef_origin_rpy:='0 0 0'
     geometry_mesh_tcp_xyz:='0 0 0'
     geometry_mesh_tcp_rpy:='0 0 0'
@@ -214,5 +218,5 @@
     </xacro:unless>
     <joint name="${prefix}joint_eef" type="fixed">
-      <origin xyz="0 0 0" rpy="0 0 0" />
+      <origin xyz="${joint_eef_origin_xyz}" rpy="${joint_eef_origin_rpy}" />
       <parent link="${prefix}link${dof}" />
       <child link="${prefix}link_eef" />
@@ -260,4 +264,5 @@
         geometry_mesh_filename="${geometry_mesh_filename}"
         geometry_mesh_origin_xyz="${geometry_mesh_origin_xyz}" geometry_mesh_origin_rpy="${geometry_mesh_origin_rpy}"
+        geometry_origin_xyz="${geometry_origin_xyz}" geometry_origin_rpy="${geometry_origin_rpy}"
         geometry_mesh_tcp_xyz="${geometry_mesh_tcp_xyz}" geometry_mesh_tcp_rpy="${geometry_mesh_tcp_rpy}"
       />
